Commit message: change color and bugs

File: dh_ag95_description/urdf/ag95.xacro (robot description, xacro)
@@ -8,11 +8,8 @@
     <xacro:dh_ag95_gripper
         prefix=""
-        transmission_hw_interface="$(arg transmission_hw_interface)" />
+        transmission_hw_interface="$(arg transmission_hw_interface)" parent="world">
+        <origin xyz="0 0 0.1" rpy="0 0 0" />
+    </xacro:dh_ag95_gripper>
     <link name="world" />
-    <joint name="world_joint" type="fixed">
-        <origin xyz="0 0 0.1" rpy="0 0 0" />
-        <parent link="world" />
-        <child link="ag95_base_link" />
-    </joint>
     <gazebo>
         <plugin name="ros_control" filename="libgazebo_ros_control.so"></plugin>

File: dh_ag95_description/urdf/ag95_gazebo.xacro (robot description, xacro)
@@ -46,5 +46,5 @@
     </gazebo>
     <gazebo reference="${prefix}left_outer_knuckle">
-      <material>Gazebo/Grey</material>
+      <material>Gazebo/Black</material>
     </gazebo>
     <gazebo reference="${prefix}left_outer_finger">
@@ -58,5 +58,5 @@
     </gazebo>
     <gazebo reference="${prefix}right_outer_knuckle">
-      <material>Gazebo/Grey</material>
+      <material>Gazebo/Black</material>
     </gazebo>
     <gazebo reference="${prefix}right_outer_finger">
@@ -69,4 +69,10 @@
       <material>Gazebo/Black</material>
     </gazebo>
+    <gazebo reference="${prefix}left_inner_finger_pad">
+      <material>Gazebo/Grey</material>
+    </gazebo>
+    <gazebo reference="${prefix}right_inner_finger_pad">
+      <material>Gazebo/Grey</material>
+    </gazebo>
   </xacro:macro>
 </robot>

File: dh_ag95_description/urdf/ag95_macro.xacro (robot description, xacro)
@@ -28,5 +28,7 @@
             <mesh filename="package://dh_ag95_description/meshes/outer_knuckle_1.stl" scale="0.001 0.001 0.001" />
           </geometry>
-          <material name="silver" />
+          <material name="">
+            <color rgba="0.1 0.1 0.1 1" />
+          </material>
         </visual>
         <collision>
@@ -50,5 +52,7 @@
             <mesh filename="package://dh_ag95_description/meshes/outer_finger_1.stl" scale="0.001 0.001 0.001" />
           </geometry>
-          <material name="silver" />
+          <material name="">
+            <color rgba="0.1 0.1 0.1 1" />
+          </material>
         </visual>
         <collision>
@@ -72,5 +76,7 @@
             <mesh filename="package://dh_ag95_description/meshes/inner_knuckle_1.stl" scale="0.001 0.001 0.001" />
           </geometry>
-          <material name="silver" />
+          <material name="">
+            <color rgba="0.1 0.1 0.1 1" />
+          </material>
         </visual>
         <collision>
@@ -94,5 +100,7 @@
             <mesh filename="package://dh_ag95_description/meshes/inner_finger_1.stl" scale="0.001 0.001 0.001" />
           </geometry>
-          <material name="silver" />
+          <material name="">
+            <color rgba="0.792156862745098 0.819607843137255 0.933333333333333 1" />
+          </material>
         </visual>
         <collision>
@@ -117,5 +125,7 @@
             <mesh filename="package://dh_ag95_description/meshes/inner_finger_pad_1.stl" scale="0.001 0.001 0.001" />
           </geometry>
-          <material name="silver" />
+          <material name="">
+            <color rgba="0.792156862745098 0.819607843137255 0.933333333333333 1" />
+          </material>
         </visual>
         <collision>
@@ -190,5 +200,7 @@
           <mesh filename="package://dh_ag95_description/meshes/base_link.stl" scale="0.001 0.001 0.001" />
         </geometry>
-        <material name="silver" />
+        <material name="">
+          <color rgba="0.792156862745098 0.819607843137255 0.933333333333333 1" />
+        </material>
       </visual>
       <collision>
@@ -211,5 +223,7 @@
           <mesh filename="package://dh_ag95_description/meshes/gripper_body_1.stl" scale="0.001 0.001 0.001" />
         </geometry>
-        <material name="silver" />
+        <material name="">
+          <color rgba="0.1 0.1 0.1 1" />
+        </material>
       </visual>
       <collision>

Commit message: effort controller interface

File: dh_ag95_description/urdf/ag95.xacro (robot description, xacro)
@@ -4,5 +4,5 @@
     <xacro:include filename="$(find dh_ag95_description)/urdf/ag95_macro.xacro" />
     <!-- parameters -->
-    <xacro:arg name="transmission_hw_interface" default="hardware_interface/PositionJointInterface" />
+    <xacro:arg name="transmission_hw_interface" default="hardware_interface/EffortJointInterface" />
     <!-- gripper -->
     <xacro:dh_ag95_gripper

File: dh_ag95_description/urdf/ag95_gazebo.xacro (robot description, xacro)
@@ -7,6 +7,4 @@
         <mimicJoint>${prefix}left_outer_finger_joint</mimicJoint>
         <multiplier>-0.4563942</multiplier>
-        <hasPID />
-        <maxEffort>100</maxEffort>
       </plugin>
       <plugin filename="libroboticsgroup_upatras_gazebo_mimic_joint_plugin.so" name="${prefix}mimic_dh_robotics_ag95_2">
@@ -14,6 +12,4 @@
         <mimicJoint>${prefix}left_inner_knuckle_joint</mimicJoint>
         <multiplier>1.45</multiplier>
-        <!-- <hasPID/>
-        <maxEffort>100</maxEffort> -->
       </plugin>
       <plugin filename="libroboticsgroup_upatras_gazebo_mimic_joint_plugin.so" name="${prefix}mimic_dh_robotics_ag95_3">
@@ -21,6 +17,4 @@
         <mimicJoint>${prefix}left_inner_finger_joint</mimicJoint>
         <multiplier>1.46</multiplier>
-        <hasPID />
-        <maxEffort>100</maxEffort>
       </plugin>
       <plugin filename="libroboticsgroup_upatras_gazebo_mimic_joint_plugin.so" name="${prefix}mimic_dh_robotics_ag95_4">
@@ -28,6 +22,4 @@
         <mimicJoint>${prefix}right_finger_joint</mimicJoint>
         <multiplier>1</multiplier>
-        <hasPID />
-        <maxEffort>100</maxEffort>
       </plugin>
       <plugin filename="libroboticsgroup_upatras_gazebo_mimic_joint_plugin.so" name="${prefix}mimic_dh_robotics_ag95_5">
@@ -35,6 +27,4 @@
         <mimicJoint>${prefix}right_outer_finger_joint</mimicJoint>
         <multiplier>-0.4563942</multiplier>
-        <hasPID />
-        <maxEffort>100</maxEffort>
       </plugin>
       <plugin filename="libroboticsgroup_upatras_gazebo_mimic_joint_plugin.so" name="${prefix}mimic_dh_robotics_ag95_6">
@@ -42,6 +32,4 @@
         <mimicJoint>${prefix}right_inner_knuckle_joint</mimicJoint>
         <multiplier>1.45</multiplier>
-        <!-- <hasPID/>
-        <maxEffort>100</maxEffort> -->
       </plugin>
       <plugin filename="libroboticsgroup_upatras_gazebo_mimic_joint_plugin.so" name="${prefix}mimic_dh_robotics_ag95_7">
@@ -49,6 +37,4 @@
         <mimicJoint>${prefix}right_inner_finger_joint</mimicJoint>
         <multiplier>1.46</multiplier>
-        <hasPID />
-        <maxEffort>100</maxEffort>
       </plugin>
     </gazebo>
@@ -65,7 +51,4 @@
       <material>Gazebo/Black</material>
     </gazebo>
-    <gazebo reference="${prefix}left_inner_finger">
-      <material>Gazebo/Grey</material>
-    </gazebo>
     <gazebo reference="${prefix}left_inner_knuckle">
       <material>Gazebo/Black</material>
@@ -77,30 +60,13 @@
       <material>Gazebo/Black</material>
     </gazebo>
+    <gazebo reference="${prefix}right_inner_knuckle">
+      <material>Gazebo/Black</material>
+    </gazebo>
+    <gazebo reference="${prefix}left_inner_finger">
+      <material>Gazebo/Grey</material>
+    </gazebo>
     <gazebo reference="${prefix}right_inner_finger">
       <material>Gazebo/Grey</material>
     </gazebo>
-    <gazebo reference="${prefix}right_inner_knuckle">
-      <material>Gazebo/Black</material>
-    </gazebo>
-    <gazebo reference="${prefix}left_inner_finger_pad">
-      <material>Gazebo/Grey</material>
-      <mu1>1000000</mu1>
-      <mu2>1000000</mu2>
-      <kp>100000000.0</kp>
-      <kd>10000000.0</kd>
-      <maxVel>0</maxVel>
-      <minDepth>0.001</minDepth>
-      <maxVel>0</maxVel>
-    </gazebo>
-    <gazebo reference="${prefix}right_inner_finger_pad">
-      <material>Gazebo/Grey</material>
-      <mu1>1000000</mu1>
-      <mu2>1000000</mu2>
-      <kp>100000000.0</kp>
-      <kd>10000000.0</kd>
-      <maxVel>0</maxVel>
-      <minDepth>0.001</minDepth>
-      <maxVel>0</maxVel>
-    </gazebo>
   </xacro:macro>
 </robot>

File: dh_ag95_description/urdf/ag95_macro.xacro (robot description, xacro)
@@ -151,5 +151,5 @@
         <child link="${prefix}${fingerprefix}_outer_finger" />
         <axis xyz="-0.0 1.0 0.0" />
-        <limit lower="${-0.29665623-0.01}" upper="0.01" velocity="0.5" effort="1000" />
+        <limit lower="${-0.29665623-0.01}" upper="0.01" velocity="0.5" effort="10" />
         <mimic joint="${prefix}finger_joint" multiplier="-0.4563942" offset="0" />
       </joint>
@@ -161,5 +161,5 @@
         <child link="${prefix}${fingerprefix}_inner_knuckle" />
         <axis xyz="0.0 -1.0 -0.0" />
-        <limit lower="-0.01" upper="${0.9425 + 0.01}" velocity="0.5" effort="1000" />
+        <limit lower="-0.01" upper="${0.9425 + 0.01}" velocity="0.5" effort="10" />
         <mimic joint="${prefix}finger_joint" multiplier="1.45" offset="0" />
       </joint>
@@ -171,5 +171,5 @@
         <child link="${prefix}${fingerprefix}_inner_finger" />
         <axis xyz="-0.0 1.0 0.0" />
-        <limit lower="-0.01" upper="${0.949 + 0.01}" velocity="0.5" effort="1000" />
+        <limit lower="-0.01" upper="${0.949 + 0.01}" velocity="0.5" effort="10" />
         <mimic joint="${prefix}finger_joint" multiplier="1.46" offset="0" />
       </joint>
@@ -247,5 +247,5 @@
       <child link="${prefix}left_outer_knuckle" />
       <axis xyz="0.0 -1.0 -0.0" />
-      <limit lower="0.0" upper="0.65" velocity="0.5" effort="1000" />
+      <limit lower="0.0" upper="0.65" velocity="0.5" effort="10" />
     </joint>
     <!-- right finger -->
@@ -257,5 +257,5 @@
       <child link="${prefix}right_outer_knuckle" />
       <axis xyz="0.0 -1.0 -0.0" />
-      <limit lower="-0.01" upper="0.66" velocity="0.5" effort="1000" />
+      <limit lower="-0.01" upper="0.66" velocity="0.5" effort="10" />
       <mimic joint="${prefix}finger_joint" multiplier="1" offset="0" />
     </joint>
