Commit message: much improved closed loop joints, 4 bar lift style

File: dh_ag95_description/urdf/ag95_gazebo.xacro (robot description, xacro)
@@ -2,71 +2,46 @@
 <robot xmlns:xacro="http://ros.org/wiki/xacro">
   <xacro:macro name="ag95_gazebo" params="prefix">
+    <!-- Mimic joint plugin -->
     <gazebo>
-      <plugin filename="libroboticsgroup_upatras_gazebo_mimic_joint_plugin.so" name="${prefix}mimic_dh_robotics_ag95_1">
-        <joint>${prefix}finger_joint</joint>
-        <mimicJoint>${prefix}left_outer_finger_joint</mimicJoint>
-        <multiplier>-0.4563942</multiplier>
-      </plugin>
-      <plugin filename="libroboticsgroup_upatras_gazebo_mimic_joint_plugin.so" name="${prefix}mimic_dh_robotics_ag95_2">
-        <joint>${prefix}finger_joint</joint>
-        <mimicJoint>${prefix}left_inner_knuckle_joint</mimicJoint>
-        <multiplier>1.45</multiplier>
-      </plugin>
       <plugin filename="libroboticsgroup_upatras_gazebo_mimic_joint_plugin.so" name="${prefix}mimic_dh_robotics_ag95_3">
-        <joint>${prefix}finger_joint</joint>
-        <mimicJoint>${prefix}left_inner_finger_joint</mimicJoint>
-        <multiplier>1.46</multiplier>
-      </plugin>
-      <plugin filename="libroboticsgroup_upatras_gazebo_mimic_joint_plugin.so" name="${prefix}mimic_dh_robotics_ag95_4">
-        <joint>${prefix}finger_joint</joint>
-        <mimicJoint>${prefix}right_finger_joint</mimicJoint>
+        <joint>${prefix}left_outer_knuckle_joint</joint>
+        <mimicJoint>${prefix}right_outer_knuckle_joint</mimicJoint>
         <multiplier>1</multiplier>
-      </plugin>
-      <plugin filename="libroboticsgroup_upatras_gazebo_mimic_joint_plugin.so" name="${prefix}mimic_dh_robotics_ag95_5">
-        <joint>${prefix}finger_joint</joint>
-        <mimicJoint>${prefix}right_outer_finger_joint</mimicJoint>
-        <multiplier>-0.4563942</multiplier>
-      </plugin>
-      <plugin filename="libroboticsgroup_upatras_gazebo_mimic_joint_plugin.so" name="${prefix}mimic_dh_robotics_ag95_6">
-        <joint>${prefix}finger_joint</joint>
-        <mimicJoint>${prefix}right_inner_knuckle_joint</mimicJoint>
-        <multiplier>1.45</multiplier>
-      </plugin>
-      <plugin filename="libroboticsgroup_upatras_gazebo_mimic_joint_plugin.so" name="${prefix}mimic_dh_robotics_ag95_7">
-        <joint>${prefix}finger_joint</joint>
-        <mimicJoint>${prefix}right_inner_finger_joint</mimicJoint>
-        <multiplier>1.46</multiplier>
+        <hasPID/>
       </plugin>
     </gazebo>
-    <gazebo reference="${prefix}ag95_base_link">
-      <material>Gazebo/Grey</material>
-    </gazebo>
-    <gazebo reference="${prefix}ag95_body">
-      <material>Gazebo/Black</material>
-    </gazebo>
-    <gazebo reference="${prefix}left_outer_knuckle">
-      <material>Gazebo/Black</material>
-    </gazebo>
-    <gazebo reference="${prefix}left_outer_finger">
-      <material>Gazebo/Black</material>
-    </gazebo>
-    <gazebo reference="${prefix}left_inner_knuckle">
-      <material>Gazebo/Black</material>
-    </gazebo>
-    <gazebo reference="${prefix}right_outer_knuckle">
-      <material>Gazebo/Black</material>
-    </gazebo>
-    <gazebo reference="${prefix}right_outer_finger">
-      <material>Gazebo/Black</material>
-    </gazebo>
-    <gazebo reference="${prefix}right_inner_knuckle">
-      <material>Gazebo/Black</material>
-    </gazebo>
-    <gazebo reference="${prefix}left_inner_finger">
-      <material>Gazebo/Grey</material>
-    </gazebo>
-    <gazebo reference="${prefix}right_inner_finger">
-      <material>Gazebo/Grey</material>
-    </gazebo>
+    <!-- Gazebo Link Properties -->
+    <xacro:macro name="ag95_gazebo_link_properties" params="reference material">
+      <gazebo reference="${reference}">
+        <material>${material}</material>
+        <kp>1000000.0</kp>
+        <kd>1.0</kd>
+        <mu1>1.16</mu1>
+        <mu2>1.16</mu2>
+        <maxVel>0.0</maxVel>
+        <minDepth>0.003</minDepth>
+      </gazebo>
+    </xacro:macro>
+    <xacro:ag95_gazebo_link_properties reference="${prefix}ag95_base_link" material="Gazebo/Grey"/>
+    <xacro:ag95_gazebo_link_properties reference="${prefix}ag95_body" material="Gazebo/Black"/>
+    <xacro:ag95_gazebo_link_properties reference="${prefix}left_outer_knuckle" material="Gazebo/Black"/>
+    <xacro:ag95_gazebo_link_properties reference="${prefix}left_inner_knuckle" material="Gazebo/Black"/>
+    <xacro:ag95_gazebo_link_properties reference="${prefix}left_finger" material="Gazebo/Grey"/>
+    <xacro:ag95_gazebo_link_properties reference="${prefix}right_outer_knuckle" material="Gazebo/Black"/>
+    <xacro:ag95_gazebo_link_properties reference="${prefix}right_inner_knuckle" material="Gazebo/Black"/>
+    <xacro:ag95_gazebo_link_properties reference="${prefix}right_finger" material="Gazebo/Grey"/>
+    <xacro:macro name="ag95_gazebo_joint_properties" params="reference">
+      <gazebo reference="${reference}">
+        <implicitSpringDamper>true</implicitSpringDamper>
+      </gazebo>
+    </xacro:macro>
+    <xacro:ag95_gazebo_joint_properties reference="${prefix}left_outer_knuckle_joint"/>
+    <xacro:ag95_gazebo_joint_properties reference="${prefix}left_finger_joint"/>
+    <xacro:ag95_gazebo_joint_properties reference="${prefix}left_inner_knuckle_joint"/>
+    <xacro:ag95_gazebo_joint_properties reference="${prefix}left_inner_knuckle_to_finger_joint"/>
+    <xacro:ag95_gazebo_joint_properties reference="${prefix}right_outer_knuckle_joint"/>
+    <xacro:ag95_gazebo_joint_properties reference="${prefix}right_finger_joint"/>
+    <xacro:ag95_gazebo_joint_properties reference="${prefix}right_inner_knuckle_joint"/>
+    <xacro:ag95_gazebo_joint_properties reference="${prefix}right_inner_knuckle_to_finger_joint"/>
   </xacro:macro>
 </robot>
