Commit message: remove pgc140

File: dh_ag95_description/urdf/ag95_macro.xacro (robot description, xacro)
@@ -6,12 +6,12 @@
     prefix
     parent
-    transmission_hw_interface:=hardware/interface/EffortJointInterface
+    transmission_hw_interface:=hardware_interface/EffortJointInterface
     *origin"
   >
     <!-- Add URDF transmission elements (for ros_control) -->
-    <xacro:ag95_transmission prefix="${prefix}" hw_interface="${transmission_hw_interface}"/>
+    <xacro:ag95_transmission prefix="${prefix}" hw_interface="${transmission_hw_interface}" />
     <xacro:ag95_gazebo prefix="${prefix}" />
     <material name="silver">
-      <color rgba="0.700 0.700 0.700 1.000"/>
+      <color rgba="0.700 0.700 0.700 1.000" />
     </material>
     <!-- fingers links macros -->
@@ -236,8 +236,8 @@
     </joint>
     <!-- right finger -->
-    <xacro:finger_joints prefix="${prefix}" fingerprefix="right" reflect="-1.0"/>
-    <xacro:finger_links prefix="${prefix}" fingerprefix="right"/>
+    <xacro:finger_joints prefix="${prefix}" fingerprefix="right" reflect="-1.0" />
+    <xacro:finger_links prefix="${prefix}" fingerprefix="right" />
     <joint name="${prefix}right_finger_joint" type="revolute">
-      <origin xyz="${0.0565 - 0.032} ${-0.0005+0.02948} 0.09116" rpy="0 ${37.211*pi/180} ${pi}"/>
+      <origin xyz="${0.0565 - 0.032} ${-0.0005+0.02948} 0.09116" rpy="0 ${37.211*pi/180} ${pi}" />
       <parent link="${prefix}ag95_body" />
       <child link="${prefix}right_outer_knuckle" />
@@ -247,8 +247,8 @@
     </joint>
     <joint name="${prefix}gripper_base_joint" type="fixed">
-      <parent link="${parent}"/>
-      <child link="${prefix}ag95_base_link"/>
-      <xacro:insert_block name="origin"/>
-  </joint>
+      <parent link="${parent}" />
+      <child link="${prefix}ag95_base_link" />
+      <xacro:insert_block name="origin" />
+    </joint>
   </xacro:macro>
 </robot>

Commit message: changed body mass and improved collision meshes. gripping very good!

File: dh_ag95_description/urdf/ag95_macro.xacro (robot description, xacro)
@@ -15,5 +15,5 @@
     <xacro:property name="lower_limit" value="0" />
     <xacro:property name="upper_limit" value="0.93" />
-    <xacro:property name="max_effort" value="10.0" />
+    <xacro:property name="max_effort" value="50.0" />
     <xacro:property name="max_velocity" value="1.0" />
     <!-- fingers links macros -->
@@ -25,4 +25,9 @@
           <inertia ixx="1e-06" iyy="1.7e-05" izz="1.7e-05" ixy="0.0" iyz="0.0" ixz="-0.0" />
         </inertial>
+        <!-- <inertial>
+          <origin xyz="0.027678515816713697 0.008750002359538555 -4.432690447753185e-07" rpy="0 0 0" />
+          <mass value="${0.0589066057773107*0.44684369179}" />
+          <inertia ixx="${1e-06*0.44684369179}" iyy="${1.7e-05*0.44684369179}" izz="${1.7e-05*0.44684369179}" ixy="${0.0*0.44684369179}" iyz="${0.0*0.44684369179}" ixz="${-0.0*0.44684369179}" />
+        </inertial> -->
         <visual>
           <origin xyz="-0.036673 0.00875 -0.098336" rpy="0 0 0" />
@@ -38,5 +43,5 @@
           <origin xyz="-0.036673 0.00875 -0.098336" rpy="0 0 0" />
           <geometry>
-            <mesh filename="package://dh_ag95_description/meshes/visual/outer_knuckle.stl"
+            <mesh filename="package://dh_ag95_description/meshes/collision/outer_knuckle.stl"
               scale="0.001 0.001 0.001" />
           </geometry>
@@ -51,4 +56,9 @@
           <inertia ixx="3.7e-05" iyy="1.7e-05" izz="2.1e-05" ixy="0.0" iyz="-0.0" ixz="0.0" />
         </inertial>
+        <!-- <inertial>
+          <origin xyz="-0.001773347637755853 0.025399999999162655 0.028950024725163018" rpy="0 0 0" />
+          <mass value="${0.07116672022913799*0.44684369179}" />
+          <inertia ixx="${3.7e-05*0.44684369179}" iyy="${1.7e-05*0.44684369179}" izz="${2.1e-05*0.44684369179}" ixy="${0.0*0.44684369179}" iyz="${-0.0*0.44684369179}" ixz="${0.0*0.44684369179}" />
+        </inertial> -->
         <visual>
           <origin xyz="-0.016 0.0254 -0.10586" rpy="0 0 0" />
@@ -64,5 +74,5 @@
           <origin xyz="-0.016 0.0254 -0.10586" rpy="0 0 0" />
           <geometry>
-            <mesh filename="package://dh_ag95_description/meshes/visual/inner_knuckle.stl"
+            <mesh filename="package://dh_ag95_description/meshes/collision/inner_knuckle.stl"
               scale="0.001 0.001 0.001" />
           </geometry>
@@ -77,4 +87,9 @@
           <inertia ixx="2e-06" iyy="4e-06" izz="3e-06" ixy="0.0" iyz="-0.0" ixz="1e-06" />
         </inertial>
+        <!-- <inertial>
+          <origin xyz="-0.013763205176003518 0.008750002316393751 0.007315452388518454" rpy="0 0 0" />
+          <mass value="${0.035304126564626004*0.14953484502}" />
+          <inertia ixx="${2e-06*0.14953484502}" iyy="${4e-06*0.14953484502}" izz="${3e-06*0.14953484502}" ixy="${0.0*0.14953484502}" iyz="${-0.0*0.14953484502}" ixz="${1e-06*0.14953484502}" />
+        </inertial> -->
         <visual>
           <origin xyz="-0.091673 0.00875 -0.098336" rpy="0 0 0" />
@@ -90,5 +105,5 @@
           <origin xyz="-0.091673 0.00875 -0.098336" rpy="0 0 0" />
           <geometry>
-            <mesh filename="package://dh_ag95_description/meshes/visual/finger.stl"
+            <mesh filename="package://dh_ag95_description/meshes/collision/finger.stl"
               scale="0.001 0.001 0.001" />
           </geometry>
@@ -104,4 +119,10 @@
           <inertia ixx="5e-06" iyy="4e-06" izz="2e-06" ixy="-0.0" iyz="0.0" ixz="0.0" />
         </inertial>
+        <!-- <inertial>
+          <origin xyz="-0.0022695421476374017 2.3166990085415594e-09 0.00779073905191241"
+            rpy="0 0 0" />
+          <mass value="${0.047823655444711066*0.14953484502}" />
+          <inertia ixx="${5e-06*0.14953484502}" iyy="${4e-06*0.14953484502}" izz="${2e-06*0.14953484502}" ixy="${-0.0*0.14953484502}" iyz="${0.0*0.14953484502}" ixz="${0.0*0.14953484502}" />
+        </inertial> -->
         <visual>
           <origin xyz="-0.0705 -0.0 -0.12056" rpy="0 0 0" />
@@ -117,5 +138,5 @@
           <origin xyz="-0.0705 -0.0 -0.12056" rpy="0 0 0" />
           <geometry>
-            <mesh filename="package://dh_ag95_description/meshes/visual/finger_pad.stl"
+            <mesh filename="package://dh_ag95_description/meshes/collision/finger_pad.stl"
               scale="0.001 0.001 0.001" />
           </geometry>
@@ -161,5 +182,6 @@
           <pose> -0.020673 0 0.007524 0 0 0</pose>
           <axis>
-            <xyz>0 0 1</xyz>
+            <xyz>0 1 0</xyz>
+            <use_parent_model_frame>false</use_parent_model_frame>
           </axis>
           <parent>${prefix}${fingerprefix}_inner_knuckle</parent>
@@ -184,8 +206,13 @@
     <!-- base link flange -->
     <link name="${prefix}ag95_base_link">
-      <inertial>
+      <!-- <inertial>
         <origin xyz="7.892486664218268e-13 9.73814800116557e-05 0.0030311891257515876" rpy="0 0 0" />
         <mass value="0.18321316702693136" />
         <inertia ixx="4e-05" iyy="0.000121" izz="0.000158" ixy="0.0" iyz="0.0" ixz="-0.0" />
+      </inertial> -->
+      <inertial>
+        <origin xyz="7.892486664218268e-13 9.73814800116557e-05 0.0030311891257515876" rpy="0 0 0" />
+        <mass value="${0.18321316702693136*0.291227699}" />
+        <inertia ixx="${4e-05*0.291227699}" iyy="${0.000121*0.291227699}" izz="${0.000158*0.291227699}" ixy="${0.0*0.291227699}" iyz="${0.0*0.291227699}" ixz="${-0.0*0.291227699}" />
       </inertial>
       <visual>
@@ -202,5 +229,5 @@
         <origin xyz="0 0 0" rpy="0 0 0" />
         <geometry>
-          <mesh filename="package://dh_ag95_description/meshes/visual/base_link.stl"
+          <mesh filename="package://dh_ag95_description/meshes/collision/base_link.stl"
             scale="0.001 0.001 0.001" />
         </geometry>
@@ -209,8 +236,13 @@
     <!-- main body of gripper -->
     <link name="${prefix}ag95_body">
-      <inertial>
+      <!-- <inertial>
         <origin xyz="0.040363309423792425 0.014263796342398428 0.04377145101823153" rpy="0 0 0" />
         <mass value="2.681074820833332" />
         <inertia ixx="0.003857" iyy="0.004463" izz="0.001562" ixy="-3e-06" iyz="-2e-06" ixz="-9e-06" />
+      </inertial> -->
+      <inertial>
+        <origin xyz="0.040363309423792425 0.014263796342398428 0.04377145101823153" rpy="0 0 0" />
+        <mass value="${2.681074820833332*0.291227699}" />
+        <inertia ixx="${0.003857*0.291227699}" iyy="${0.004463*0.291227699}" izz="${0.001562*0.291227699}" ixy="${-3e-06*0.291227699}" iyz="${-2e-06*0.291227699}" ixz="${-9e-06*0.291227699}" />
       </inertial>
       <visual>
@@ -227,5 +259,5 @@
         <origin xyz="0.0405 0.0143 -0.0147" rpy="0 0 0" />
         <geometry>
-          <mesh filename="package://dh_ag95_description/meshes/visual/gripper_body.stl"
+          <mesh filename="package://dh_ag95_description/meshes/collision/gripper_body.stl"
             scale="0.001 0.001 0.001" />
         </geometry>

Commit message: update ag95_macro.xacro

File: dh_ag95_description/urdf/ag95_macro.xacro (robot description, xacro)
@@ -16,5 +16,5 @@
     <xacro:property name="upper_limit" value="0.93" />
     <xacro:property name="max_effort" value="50.0" />
-    <xacro:property name="max_velocity" value="1.0" />
+    <xacro:property name="max_velocity" value="2.0" />
     <!-- fingers links macros -->
     <xacro:macro name="outer_knuckle" params="prefix fingerprefix">
